Commit message: Added resources

File: resources/fetch_description/robots/fetch.urdf (robot description, URDF)
Before this commit: robot fetch, 21 links, 20 joints
Links:
- removed link head_pan_link
- removed link head_tilt_link
Joints:
- removed joint head_pan_joint
- removed joint head_tilt_joint
